File: avr_programmer/avr_programmer.kicad_pcb (KiCad board)
At the start: 2 copper layers, 76.2 x 77.5 mm, 9 parts, among them IC1 ATMEGA168-P, P1 CONN_3X2

Commit message: Update 'avr_programmer'.
Other:
- net class Default: via_dia 1.5 -> 2.2
